File: PROTO_PCB_2022.sch (KiCad schematic (older format))
At the start: 14 parts, among them J1 ECU_EN_CONNECTION, J2 SMALL_12V_BATTERY_CONNECTOR, J3 12V_EXTRA, J4 ECU_EN_CONNECTION, K1 RT214012, K2 RT214012, U1 ATtiny85-20MU

Commit message: Fixed connectors, removed MCU, final first draft
Parts:
- removed J4: ECU_EN_CONNECTION, Connector_Molex:Molex_Micro-Fit_3.0_43650-0315_1x03_P3.00mm_Vertical, symbol Connector_Generic:Conn_01x03
- removed U1: ATtiny85-20MU, Package_DFN_QFN:QFN-20-1EP_4x4mm_P0.5mm_EP2.6x2.6mm, symbol MCU_Microchip_ATtiny:ATtiny85-20MU
- added HORN_EN?: Conn_?, Connector_Molex:Molex_Micro-Fit_3.0_43045-0218_2x01-1MP_P3.00mm_Vertical, symbol PROTO_PCB_2022-rescue:B2B-PH-K-S_LF__SN_-dk_Rectangular-Connectors-Headers-Male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
- BRAKELIGHTS_EN1, HORN_EN1, STARTER_MOTOR_EN1: footprint Connector_Molex:Molex_Micro-Fit_3.0_43045-0218_2x01-1MP_P3.00mm_Vertical -> Footprint Library:Molex_Proto_Microfit_Footprint; DigiKeyPN WM1801CT-ND -> WM10657-ND; MPN 0430450218 -> 0430450227
- J2, J3: footprint digikey-footprints:Terminal_Block_D1.3mm_P5mm -> TerminalBlock_Phoenix:TerminalBlock_Phoenix_PT-1,5-2-5.0-H_1x02_P5.00mm_Horizontal; symbol dk_Terminal-Blocks-Wire-to-Board:1935161 -> PROTO_PCB_2022-rescue:1935161-dk_Terminal-Blocks-Wire-to-Board
Connections:
- net labels added: Conn_?, ECU_POWER
- net labels removed: ECU_KEYSW_WIRE, O2_ANALOG_READING_SIGNAL
- wire segments 47 -> 46
Other:
- note removed: "3 connection-Molex: PWR (12V), GND, SIG(O2)"
- note removed: "To Do:\n1. DONE - Add Mini ATtiny85 board\n2. DONE - Add Oxygen Sensor (header)="
- note removed: "To Do:\n1. Talk to Powertrain about ECU: KEYSW, Relay and O2 Sensor\n"
- moved on the sheet: BRAKELIGHTS_MOSFET1, HORN_MOSFET1, J2, J3, R1, R2
