File: PROTO_PCB_2022.sch (KiCad schematic (older format))
At the start: 13 parts, among them J1 ECU_EN_CONNECTION, J2 SMALL_12V_BATTERY_CONNECTOR, J3 12V_EXTRA, K1 RT214012, K2 RT214012

Commit message: Updated ECU connector
Parts:
- removed HORN_EN?: Conn_?, Connector_Molex:Molex_Micro-Fit_3.0_43045-0218_2x01-1MP_P3.00mm_Vertical, symbol PROTO_PCB_2022-rescue:B2B-PH-K-S_LF__SN_-dk_Rectangular-Connectors-Headers-Male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
- J1: footprint Connector_Molex:Molex_CLIK-Mate_502386-0470_1x04-1MP_P1.25mm_Horizontal -> Connector_Molex:Molex_Micro-Fit_3.0_43650-0400_1x04_P3.00mm_Horizontal; DigikeyPN WM4948CT-ND -> WM1862-ND; MPN 5023860470 -> 0436500400
- Q1: renamed from HORN_MOSFET1; value Q1 -> HORN_MOSFET1
- Q2: renamed from BRAKELIGHTS_MOSFET1; value Q3 -> BRAKELIGHTS_MOSFET1
Other:
- moved on the sheet: J3

Commit message: replaced 4 pin ECU_EN with 3 2 pin connectors, removed ECU relay and set ECU kill switches in series
Parts:
- removed J1: ECU_EN_CONNECTION, Connector_Molex:Molex_Micro-Fit_3.0_43650-0400_1x04_P3.00mm_Horizontal, symbol Connector_Generic:Conn_01x04
- removed K1: RT214012, Relay_THT:Relay_SPDT_Schrack-RT1-FormC_RM5mm, symbol Relay:RT314A12
- added J?: Conn_01x02_Male, symbol Connector:Conn_01x02_Male
- added J?: ECU_EN_CONNECTON_1, Connector_Molex:Molex_Micro-Fit_3.0_43650-0215_1x02_P3.00mm_Vertical, symbol Connector_Generic:Conn_01x02
- added J?: ECU_EN_CONECTION_2, Connector_Molex:Molex_Micro-Fit_3.0_43650-0215_1x02_P3.00mm_Vertical, symbol Connector_Generic:Conn_01x02
- added J?: ECU_EN_CONECTION_3, Connector_Molex:Molex_Micro-Fit_3.0_43650-0215_1x02_P3.00mm_Vertical, symbol Connector_Generic:Conn_01x02
Connections:
- net labels added: ECU_KILL_EN_TOGGLESWITCH_1A, ECU_KILL_EN_TOGGLESWITCH_1B, ECU_KILL_EN_TOGGLESWITCH_2A, ECU_KILL_EN_TOGGLESWITCH_2B, ECU_KILL_EN_TOGGLESWITCH_3A, ECU_KILL_EN_TOGGLESWITCH_3B
- wire segments 46 -> 47
Other:
- note removed: "When Coil is Powered: ECU is not powered - Relay is disconnected\nWhen Coil is Not Powered: ECU is powered - Relay is connected\n> NORMALLY ON RELAY, 5A ON CONTACTS\n\n\n"
- moved on the sheet: BRAKELIGHTS_EN1, HORN_EN1, J2, STARTER_MOTOR_EN1

Commit message: added new TVS diodes to schematic
Parts:
- removed J?: Conn_01x02_Male, symbol Connector:Conn_01x02_Male
- added D1: HORN_D_TVS, Diode_SMD:D_SMB, symbol Device:D_TVS
- added D2: BRAKELIGHTS_D_TVS, Diode_SMD:D_SMB, symbol Device:D_TVS
- gave numbers to parts that had none: 3
Connections:
- net BRAKELIGHTS_EN_12V_SIGNAL: now also D2.1 (A1)
- net BRAKELIGHTS_PWR: now also D2.2 (A2)
- net HORN_EN_12V_SIGNAL: now also D1.2 (A2)
- net HORN_PWR: now also D1.1 (A1)
Changed lines of the file:
@@
 $EndComp
-Wire Wire Line
-	8900 3050 8900 3150
 Wire Wire Line
 	8400 2850 8400 2950
 Wire Wire Line
 	8400 3250 8400 3350
-$Comp
-L Device:Q_NMOS_DGS Q2
-U 1 1 618C50B5
-P 8800 4550
-F 0 "Q2" H 9005 4596 50  0000 L CNN
-F 1 "BRAKELIGHTS_MOSFET1" H 9005 4505 50  0000 L CNN
-F 2 "Package_TO_SOT_SMD:SOT-23" H 9000 4650 50  0001 C CNN
-F 3 "https://www.digikey.ca/en/products/detail/rohm-semiconductor/RK7002BMT116/4924083" H 8800 4550 50  0001 C CNN
-F 4 "RK7002BMT116" H 8800 4550 50  0001 C CNN "MPN"
-F 5 "RK7002BMT116CT-ND" H 8800 4550 50  0001 C CNN "DigiKeyPN"
-	1    8800 4550
-	1    0    0    -1
-$EndComp
-Wire Wire Line
-	8600 4550 8400 4550
 Wire Wire Line
 	8400 4950 8400 5100
@@
 Wire Wire Line
 	9700 3350 9650 3350
-Wire Wire Line
-	8900 4750 8900 4850
 $Comp
 L Device:R #R4
@@
 	1    9500 3350
 	0    1    1    0
-$EndComp
-$Comp
-L Device:R R2
-U 1 1 61E941D5
-P 8400 4800
-F 0 "R2" H 8470 4846 50  0000 L CNN
-F 1 "10k" H 8470 4755 50  0000 L CNN
-F 2 "Resistor_SMD:R_0805_2012Metric" V 8330 4800 50  0001 C CNN
-F 3 "https://www.yageo.com/upload/media/product/productsearch/datasheet/rchip/PYu-RC_Group_51_RoHS_L_11.pdf" H 8400 4800 50  0001 C CNN
-F 4 "RC0805FR-0710RL" H 8400 4800 50  0001 C CNN "MPN"
-F 5 "311-10.0CRCT-ND" H 8400 4800 50  0001 C CNN "DigikeyPN"
-	1    8400 4800
-	1    0    0    -1
 $EndComp
 Text Notes 1350 5750 0    50   ~ 0
@@
 	2150 3250 2300 3250
 $Comp
-L Connector:Conn_01x02_Male J?
+L Connector:Conn_01x02_Male #J6
 U 1 1 61F7B731
 P 7300 1650
-F 0 "J?" H 7408 1831 50  0000 C CNN
+F 0 "#J6" H 7408 1831 50  0000 C CNN
 F 1 "Conn_01x02_Male" H 7408 1740 50  0000 C CNN
 F 2 "" H 7300 1650 50  0001 C CNN
@@
 $EndComp
 $Comp
-L Connector_Generic:Conn_01x02 J?
+L Connector_Generic:Conn_01x02 J1
 U 1 1 61F7F680
 P 2500 2650
-F 0 "J?" H 2580 2642 50  0000 L CNN
+F 0 "J1" H 2580 2642 50  0000 L CNN
 F 1 "ECU_EN_CONNECTON_1" H 2580 2551 50  0000 L CNN
 F 2 "Connector_Molex:Molex_Micro-Fit_3.0_43650-0215_1x02_P3.00mm_Vertical" H 2500 2650 50  0001 C CNN
@@
 $EndComp
 $Comp
-L Connector_Generic:Conn_01x02 J?
+L Connector_Generic:Conn_01x02 J4
 U 1 1 61F820EC
 P 2500 2950
-F 0 "J?" H 2580 2942 50  0000 L CNN
+F 0 "J4" H 2580 2942 50  0000 L CNN
 F 1 "ECU_EN_CONECTION_2" H 2580 2851 50  0000 L CNN
 F 2 "Connector_Molex:Molex_Micro-Fit_3.0_43650-0215_1x02_P3.00mm_Vertical" H 2500 2950 50  0001 C CNN
@@
 $EndComp
 $Comp
-L Connector_Generic:Conn_01x02 J?
+L Connector_Generic:Conn_01x02 J5
 U 1 1 61F82F62
 P 2500 3250
-F 0 "J?" H 2580 3242 50  0000 L CNN
+F 0 "J5" H 2580 3242 50  0000 L CNN
 F 1 "ECU_EN_CONECTION_3" H 2580 3151 50  0000 L CNN
 F 2 "Connector_Molex:Molex_Micro-Fit_3.0_43650-0215_1x02_P3.00mm_Vertical" H 2500 3250 50  0001 C CNN
@@
 Wire Wire Line
 	2250 5150 3150 5150
+$Comp
+L Device:Q_NMOS_DGS Q2
+U 1 1 618C50B5
+P 8800 4550
+F 0 "Q2" H 9005 4596 50  0000 L CNN
+F 1 "BRAKELIGHTS_MOSFET1" H 9005 4505 50  0000 L CNN
+F 2 "Package_TO_SOT_SMD:SOT-23" H 9000 4650 50  0001 C CNN
+F 3 "https://www.digikey.ca/en/products/detail/rohm-semiconductor/RK7002BMT116/4924083" H 8800 4550 50  0001 C CNN
+F 4 "RK7002BMT116" H 8800 4550 50  0001 C CNN "MPN"
+F 5 "RK7002BMT116CT-ND" H 8800 4550 50  0001 C CNN "DigiKeyPN"
+	1    8800 4550
+	1    0    0    -1
+$EndComp
+Wire Wire Line
+	8600 4550 8400 4550
+$Comp
+L Device:R R2
+U 1 1 61E941D5
+P 8400 4800
+F 0 "R2" H 8470 4846 50  0000 L CNN
+F 1 "10k" H 8470 4755 50  0000 L CNN
+F 2 "Resistor_SMD:R_0805_2012Metric" V 8330 4800 50  0001 C CNN
+F 3 "https://www.yageo.com/upload/media/product/productsearch/datasheet/rchip/PYu-RC_Group_51_RoHS_L_11.pdf" H 8400 4800 50  0001 C CNN
+F 4 "RC0805FR-0710RL" H 8400 4800 50  0001 C CNN "MPN"
+F 5 "311-10.0CRCT-ND" H 8400 4800 50  0001 C CNN "DigikeyPN"
+	1    8400 4800
+	1    0    0    -1
+$EndComp
+$Comp
+L Device:D_TVS D2
+U 1 1 622E5E5E
+P 8600 4750
+F 0 "D2" V 8554 4830 50  0000 L CNN
+F 1 "BRAKELIGHTS_D_TVS" V 8645 4830 50  0000 L CNN
+F 2 "Diode_SMD:D_SMB" H 8600 4750 50  0001 C CNN
+F 3 "https://media.digikey.com/pdf/Data%20Sheets/AVX%20PDFs/Transient%20Suppression%20Diodes.pdf~" H 8600 4750 50  0001 C CNN
+	1    8600 4750
+	0    1    1    0
+$EndComp
+Wire Wire Line
+	8600 4600 8600 4550
+Connection ~ 8600 4550
+Wire Wire Line
+	8600 4900 8900 4900
+Wire Wire Line
+	8900 4750 8900 4900
+$Comp
+L Device:D_TVS D1
+U 1 1 62314A6C
+P 8600 3050
+F 0 "D1" V 8646 2970 50  0000 R CNN
+F 1 "HORN_D_TVS" V 8555 2970 50  0000 R CNN
+F 2 "Diode_SMD:D_SMB" H 8600 3050 50  0001 C CNN
+F 3 "https://media.digikey.com/pdf/Data%20Sheets/AVX%20PDFs/Transient%20Suppression%20Diodes.pdf" H 8600 3050 50  0001 C CNN
+	1    8600 3050
+	0    -1   -1   0
+$EndComp
+Wire Wire Line
+	8600 2900 8600 2850
+Connection ~ 8600 2850
+Wire Wire Line
+	8600 3200 8900 3200
+Wire Wire Line
+	8900 3050 8900 3200
 $EndSCHEMATC

Commit message: Draft PCB for Report Purposes
Parts:
- removed J1: ECU_EN_CONNECTON_1, Connector_Molex:Molex_Micro-Fit_3.0_43650-0215_1x02_P3.00mm_Vertical, symbol Connector_Generic:Conn_01x02
- removed J4: ECU_EN_CONECTION_2, Connector_Molex:Molex_Micro-Fit_3.0_43650-0215_1x02_P3.00mm_Vertical, symbol Connector_Generic:Conn_01x02
- removed J5: ECU_EN_CONECTION_3, Connector_Molex:Molex_Micro-Fit_3.0_43650-0215_1x02_P3.00mm_Vertical, symbol Connector_Generic:Conn_01x02
- added J10: VESC_EN_SIGNAL, Footprint Library:Molex_Proto_Microfit_Footprint, symbol PROTO_PCB_2022-rescue:B2B-PH-K-S_LF__SN_-dk_Rectangular-Connectors-Headers-Male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
- added J11: BRAKELIGHTS_PWR_OUT, Footprint Library:Molex_Proto_Microfit_Footprint, symbol PROTO_PCB_2022-rescue:B2B-PH-K-S_LF__SN_-dk_Rectangular-Connectors-Headers-Male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
- added J12: HORN_PWR_OUT, Footprint Library:Molex_Proto_Microfit_Footprint, symbol PROTO_PCB_2022-rescue:B2B-PH-K-S_LF__SN_-dk_Rectangular-Connectors-Headers-Male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
- added J6: ECU_POWER_DIST, TerminalBlock_Phoenix:TerminalBlock_Phoenix_PT-1,5-2-5.0-H_1x02_P5.00mm_Horizontal, symbol PROTO_PCB_2022-rescue:1935161-dk_Terminal-Blocks-Wire-to-Board
- added J7: ECU_KILL_1, Footprint Library:Molex_Proto_Microfit_Footprint, symbol PROTO_PCB_2022-rescue:B2B-PH-K-S_LF__SN_-dk_Rectangular-Connectors-Headers-Male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
- added J8: ECU_KILL_2, Footprint Library:Molex_Proto_Microfit_Footprint, symbol PROTO_PCB_2022-rescue:B2B-PH-K-S_LF__SN_-dk_Rectangular-Connectors-Headers-Male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
- added J9: ECU_KILL_3, Footprint Library:Molex_Proto_Microfit_Footprint, symbol PROTO_PCB_2022-rescue:B2B-PH-K-S_LF__SN_-dk_Rectangular-Connectors-Headers-Male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
- J1: renamed from HORN_EN1; value Conn_? -> HORN_EN1
- J2: renamed from BRAKELIGHTS_EN1; value Conn_? -> BRAKELIGHTS_EN1
- J3: renamed from STARTER_MOTOR_EN1; value Conn_? -> STARTER_MOTOR_EN
- J4: renamed from J2; value SMALL_12V_BATTERY_CONNECTOR -> 12V_BATT1
- renumbered D2 to D1, D1 to D2, J3 to J5, K2 to K1, Q2 to Q1, Q1 to Q2, R2 to R1, R1 to R2
Connections:
- net BRAKELIGHTS_PWR is gone; now on net GND: D1.2 (A2), Q1.3 (S)
- net HORN_PWR is gone; now on net GND: D2.1 (A1), Q2.3 (S)
- net ECU_KILL_EN_TOGGLESWITCH_1A: now also J7.2; no longer Q1.1 (D), Q2.1 (D)
- net ECU_KILL_EN_TOGGLESWITCH_1B: now also J7.1, J8.2
- net ECU_KILL_EN_TOGGLESWITCH_2B: now also J8.1, J9.2
- net ECU_KILL_EN_TOGGLESWITCH_3B: now also J6.2, J9.1
- net GND: now also J10.1, J11.1, J12.1, J6.1
- net VESC_POWER_CONNECTION renamed VESC_EN_SIGNAL
- net VESC_EN_SIGNAL: now also J10.2
- new net BRAKELIGHTS_PWR_OUT: J11.2, Q1.1 (D)
- new net HORN_PWR_OUT: J12.2, Q2.1 (D)
Other:
- note removed: "SHOULD WE SEPARATE SIGNAL_12V FROM POWER_12V?"
- note removed: "Starter Motor is normally not connected - only powered when push button is being pressed"
- moved on the sheet: D1, D2, J1, J2, J3, J4, J5, Q1, Q2, R1, R2

Commit message: second version
Parts:
- removed J11: BRAKELIGHTS_PWR_OUT, Footprint Library:Molex_Proto_Microfit_Footprint, symbol PROTO_PCB_2022-rescue:B2B-PH-K-S_LF__SN_-dk_Rectangular-Connectors-Headers-Male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
- removed J12: HORN_PWR_OUT, Footprint Library:Molex_Proto_Microfit_Footprint, symbol PROTO_PCB_2022-rescue:B2B-PH-K-S_LF__SN_-dk_Rectangular-Connectors-Headers-Male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
- removed K1: RT214012, Relay_THT:Relay_SPDT_Schrack-RT1-FormC_RM5mm, symbol Relay:RT314A12
- added H1, H2: MountingHole, MountingHole:MountingHole_2.7mm_M2.5, symbol Mechanical:MountingHole
- added J3: BRAKELIGHTS_CONN, TerminalBlock_Phoenix:TerminalBlock_Phoenix_PT-1,5-2-5.0-H_1x02_P5.00mm_Horizontal, symbol PROTO_PCB_2022-rescue:1935161-dk_Terminal-Blocks-Wire-to-Board
- added J6: HORN_CONN, TerminalBlock_Phoenix:TerminalBlock_Phoenix_PT-1,5-2-5.0-H_1x02_P5.00mm_Horizontal, symbol PROTO_PCB_2022-rescue:1935161-dk_Terminal-Blocks-Wire-to-Board
- added R3: 10k, Resistor_SMD:R_0603_1608Metric, symbol Device:R
- added U1: LD1117S50TR_SOT223, Package_TO_SOT_SMD:SOT-223-3_TabPin2, symbol Regulator_Linear:LD1117S50TR_SOT223
- renumbered D2 to D1, D1 to D2, J8 to J10, J9 to J11, J5 to J12, J3 to J4, J10 to J5, J4 to J7, J6 to J8, J7 to J9, Q2 to Q1, Q1 to Q2, R2 to R1, R1 to R2
Connections:
- net GND: now also R3.2, U1.1 (GND); no longer J1.1, J2.1, J4.1, J5.1
- net BRAKELIGHTS_EN_12V_SIGNAL renamed BRAKELIGHTS_EN_5V
- net BRAKELIGHTS_EN_5V: now also J2.1; no longer J2.2
- net BRAKELIGHTS_PWR_OUT renamed BRAKELIGHTS_GND
- net BRAKELIGHTS_GND: now also J3.1
- net ECU_KILL_EN_TOGGLESWITCH_1A renamed +12V
- net +12V: now also J3.2, J6.2, U1.3 (VI)
- net HORN_EN_12V_SIGNAL renamed HORN_EN_5V
- net HORN_EN_5V: now also J1.1; no longer J1.2
- net HORN_PWR_OUT renamed HORN_GND
- net HORN_GND: now also J6.1
- net STARTER_EN_PUSHBUTTON renamed +5V
- net +5V: now also J1.2, J2.2, U1.2 (VO)
- net VESC_EN_SIGNAL renamed VESC_EN_5V
- net VESC_EN_5V: now also J4.1
- new net: J5.1, R3.1
Other:
- note added: "MOUNTING HOLES"
- note added: "POWER AND 12V TO 5V REGULATOR"
- note added: "POWER, HORN, BRAKELIGHTS"
- note added: "STARTER, ECU\n"
- note added: "does this resistor make sense?\nthe intention was to dissipate anything remaining"
- note added: "then by that logic do we need one here too?"
- note removed: "HORN AND BRAKELIGHTS"
- note removed: "POWER AND CONNECTIONS\n"
- note removed: "STARTER AND ECU\n"
- moved on the sheet: D1, D2, J1, J10, J11, J12, J2, J4, J5, J7, J8, J9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

Commit message: second version
Connections:
- net +12V: no longer J12.2
- net GND: now also J5.1; no longer J12.1
- net VESC_EN_5V: now also R3.1
Other:
- note added: "DOES VESC HAVE ITS OWN PULL DOWN RESISTOR?\ndoes this resistor make sense?\nthe intention was to dissipate anything remaining"
- note added: "HORN, BRAKELIGHTS"
- note added: "add diode"
- note added: "add pads for 5v and 12v\nadd LED lights to show when buttons are being pressed\nchange to horizontal molex connectors\ncurrent sense probe for oscilloscope?"
- note added: "remove tvs\nchange mosfet"
- note removed: "POWER, HORN, BRAKELIGHTS"
- note removed: "does this resistor make sense?\nthe intention was to dissipate anything remaining"
- note removed: "then by that logic do we need one here too?"
- moved on the sheet: J1, J12, J2, J3, J4, J5, J6, J8, R3
