File: PROTO_PCB.kicad_sch (KiCad schematic)
At the start: 33 parts, among them J1 12V_IN, J10 12V_AUX, J12 VESC_START, J2 Ethernet connector, J3 SW_KILL_LEFT, J4 SW_KILL_RIGHT, J5 12V_ECU, J8 12V_TEL, J9 12V_HORN, Q1 MOSFET_ECU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

Commit message: VESC connector labels
Parts:
- Q1: value MOSFET_ECU -> (none); footprint Package_TO_SOT_SMD:TO-252-3_TabPin2 -> (none)
Changed lines of the file:
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@@
       (effects (font (size 1.27 1.27)) (justify left))
     )
-    (property "Value" "MOSFET_ECU" (id 1) (at 77.5716 135.763 0)
+    (property "Value" "" (id 1) (at 77.5716 135.763 0)
       (effects (font (size 1.27 1.27)) (justify left))
     )
-    (property "Footprint" "Package_TO_SOT_SMD:TO-252-3_TabPin2" (id 2) (at 77.47 132.08 0)
+    (property "Footprint" "" (id 2) (at 77.47 132.08 0)
       (effects (font (size 1.27 1.27)) hide)
     )
